Commit message: added lidar imu and odom to urdf file

File: urdf/swebot.urdf (robot description, URDF)
Before this commit: robot swebot, 6 links, 5 joints
Links:
- added link imu_link, mass 0.01
- added link lidar_link, mass 0.1; visual cylinder length=0.04 radius=0.035
- link body: mass 0.0114518 -> 2.0; geometry collision box size=0.22 0.42 0.15; visual mesh filename=package://swebot/meshes/body.stl scale=1 1 1
- link caster_body: mass 9.7853e-05 -> 0.05; geometry visual mesh filename=package://swebot/meshes/caster_body.stl scale=1 1 1
- link caster_wheel: mass 0.00019635 -> 0.05; geometry collision sphere radius=0.05; visual mesh filename=package://swebot/meshes/caster_wheel.stl scale=1 1 1
- link left_wheel: mass 0.0015708 -> 0.15; geometry collision cylinder length=0.05 radius=0.1; visual mesh filename=package://swebot/meshes/left_wheel.stl scale=1 1 1
- link right_wheel: mass 0.0015708 -> 0.15; geometry collision cylinder length=0.05 radius=0.1; visual mesh filename=package://swebot/meshes/right_wheel.stl scale=1 1 1
Joints:
- removed joint fixed_node_to_root_joint
- removed joint revolute_1
- removed joint revolute_2
- removed joint revolute_3
- removed joint revolute_4
- added joint base_to_body: type fixed, parent base_link, child body, origin xyz=0.323981 0 0.146 rpy=0 0 1.5708
- added joint caster_swivel_joint: type continuous, parent body, child caster_body, origin xyz=0 0.0557349 -0.0335411 rpy=0 0 0, axis 0 0 1
- added joint caster_wheel_joint: type continuous, parent caster_body, child caster_wheel, origin xyz=0 -0.0317543 -0.0625 rpy=0 0 0, axis 1 0 0
- added joint imu_joint: type fixed, parent base_link, child imu_link, origin xyz=0 0 0.15 rpy=0 0 0
- added joint left_wheel_joint: type continuous, parent body, child left_wheel, origin xyz=0.135 0.323981 -0.0460411 rpy=0 0 0, axis 1 0 0
- added joint lidar_joint: type fixed, parent base_link, child lidar_link, origin xyz=0.09 0 0.23 rpy=0 0 0
- added joint right_wheel_joint: type continuous, parent body, child right_wheel, origin xyz=-0.135 0.323981 -0.0460411 rpy=0 0 0, axis 1 0 0
